Commit message: Updated URDF for MP4 and clean comments

File: sawyer_description/urdf/sawyer.urdf (robot description, URDF)
Before this commit: robot sawyer, 19 links, 18 joints
Joints:
- joint right_j0: limit lower=-3.0503 upper=3.0503 effort=80.0 velocity=1.48 -> lower=-3.0503 upper=3.0503 effort=80.0 velocity=1.74
- joint right_j1: limit lower=-3.8183 upper=2.2824 effort=80.0 velocity=1.13 -> lower=-3.8183 upper=2.2824 effort=80.0 velocity=1.328
- joint right_j2: limit lower=-3.0514 upper=3.0514 effort=40.0 velocity=1.66 -> lower=-3.0514 upper=3.0514 effort=40.0 velocity=1.957
- joint right_j3: limit lower=-3.0514 upper=3.0514 effort=40.0 velocity=1.66 -> lower=-3.0514 upper=3.0514 effort=40.0 velocity=1.957
- joint right_j4: limit lower=-2.9842 upper=2.9842 effort=9.0 velocity=2.96 -> lower=-2.9842 upper=2.9842 effort=9.0 velocity=3.485
- joint right_j5: limit lower=-2.9842 upper=2.9842 effort=9.0 velocity=2.96 -> lower=-2.9842 upper=2.9842 effort=9.0 velocity=3.485
- joint right_j6: limit lower=-4.7104 upper=4.7104 effort=9.0 velocity=3.86 -> lower=-4.7104 upper=4.7104 effort=9.0 velocity=4.545

Commit message: Updates to default (sim) camera frame
Port updates to the default URDF camera frames, so that the tf frames are located at the
focal point instead of on the sensor. NOTE: only applies to sim robots, as physical robots
use a frame derived from manufacturing calibration.

File: sawyer_description/urdf/sawyer.urdf (robot description, URDF)
Before this commit: robot sawyer, 19 links, 18 joints
Joints:
- joint head_camera: origin xyz=0.015925 0 0.22087 rpy=-2.1293 0 -1.57079632679 -> xyz=0.0228027 0 0.216572 rpy=-2.1293 0 -1.57079632679
- joint right_hand_camera: origin xyz=0.019552 -0.033 0.0695 rpy=0 1.57079632679 0 -> xyz=0.039552 -0.033 0.0695 rpy=0 1.57079632679 0

Commit message: Added controller box URDF shapes
These shapes are optional on the URDF, but
desired by default to prevent unnecessary collisions
with the robot's base and controller. Likely they
will be made optional in a future Xacro of Sawyer's
URDF.

File: sawyer_description/urdf/sawyer.urdf (robot description, URDF)
Before this commit: robot sawyer, 19 links, 18 joints
Links:
- added link controller_box; collision box size=0.22 0.4 0.53
- added link pedestal_feet; collision box size=0.77 0.7 0.31
Joints:
- added joint controller_box_fixed: type fixed, parent base, child controller_box, origin xyz=0.0 0.0 0.0 rpy=0 0 0
- added joint pedestal_feet_fixed: type fixed, parent base, child pedestal_feet, origin xyz=0.0 0.0 0.0 rpy=0 0 0

Commit message: Updated URDF masses and collision shapes
This URDF modification contains the following changes
for the Sawyer robot:

- More accurate mass and inertial values for linkages
- Tighter collision shapes, and secondary linkages
  containing additional collision shapes

File: sawyer_description/urdf/sawyer.urdf (robot description, URDF)
Before this commit: robot sawyer, 21 links, 20 joints
Links:
- added link right_l1_2, mass 1.0E-08; collision cylinder length=0.14 radius=0.07
- added link right_l2_2, mass 1.0E-08; collision sphere radius=0.06
- added link right_l4_2, mass 1.0E-08; collision sphere radius=0.06
- link right_hand: geometry collision cylinder length=0.03 radius=0.035
- link right_l2: mass 1.7251 -> 1.745; geometry collision cylinder length=0.34 radius=0.06; visual mesh filename=package://sawyer_description/meshes/sawyer_pv/l2.DAE
- link right_l3: mass 2.4743 -> 2.5097
- link right_l4: mass 1.0433 -> 1.052926; geometry collision cylinder length=0.30 radius=0.045; visual mesh filename=package://sawyer_description/meshes/sawyer_pv/l4.DAE
- link right_l5: mass 1.5343 -> 1.5625
- link right_l6: geometry collision cylinder length=0.05 radius=0.055; visual mesh filename=package://sawyer_description/meshes/sawyer_mp1/l6.DAE
Joints:
- added joint right_j1_2: type fixed, parent right_l1, child right_l1_2, origin xyz=0 0 0 rpy=0 0 0, axis 0 0 1
- added joint right_j2_2: type fixed, parent right_l2, child right_l2_2, origin xyz=0 0 0 rpy=0 0 0, axis 0 0 1
- added joint right_j4_2: type fixed, parent right_l4, child right_l4_2, origin xyz=0 0 0 rpy=0 0 0, axis 0 0 1
- joint head_pan: limit lower=-5.1477 upper=0.9559 effort=8 velocity=1.8 -> lower=-5.0952 upper=0.9064 effort=8 velocity=1.8
- joint right_j1: limit lower=-3.8183 upper=2.2824 effort=80.0 velocity=1.328 -> lower=-3.8095 upper=2.2736 effort=80.0 velocity=1.328
- joint right_j2: limit lower=-3.0514 upper=3.0514 effort=40.0 velocity=1.957 -> lower=-3.0426 upper=3.0426 effort=40.0 velocity=1.957
- joint right_j3: limit lower=-3.0514 upper=3.0514 effort=40.0 velocity=1.957 -> lower=-3.0439 upper=3.0439 effort=40.0 velocity=1.957
- joint right_j4: limit lower=-2.9842 upper=2.9842 effort=9.0 velocity=3.485 -> lower=-2.9761 upper=2.9761 effort=9.0 velocity=3.485
- joint right_j5: limit lower=-2.9842 upper=2.9842 effort=9.0 velocity=3.485 -> lower=-2.9761 upper=2.9761 effort=9.0 velocity=3.485
- joint right_j6: limit lower=-4.7104 upper=4.7104 effort=9.0 velocity=4.545 -> lower=-4.7124 upper=4.7124 effort=9.0 velocity=4.545

Commit message: Updated for Sawyer MP4 model

File: sawyer_description/urdf/sawyer.urdf (robot description, URDF)
Before this commit: robot sawyer, 24 links, 23 joints
Links:
- link right_l4: mass 1.052926 -> 1.1136
