Commit message: Fix pedestal COM, color, and TF

File: sawyer_description/urdf/sawyer_base.gazebo.xacro (robot description, xacro)
@@ -10,4 +10,12 @@
   </gazebo -->
   <!-- Gazebo-Specific Link Properties -->
+  <link name="world"/>
+    <joint name="fixed" type="fixed">
+      <parent link="world"/>
+      <child link="base"/>
+  </joint>
+  <gazebo reference="pedestal">
+    <material>Gazebo/FlatBlack</material>
+  </gazebo>
   <gazebo reference="torso">
     <self_collide>true</self_collide>

File: sawyer_description/urdf/sawyer_base.urdf.xacro (robot description, xacro)
@@ -53,5 +53,5 @@
     </collision>
     <inertial>
-      <origin rpy="0 0 0" xyz="0 0 0"/>
+      <origin rpy="0 0 0" xyz="0 0 -0.5"/>
       <mass value="60.86397744"/>
       <inertia ixx="5.0635929" ixy="0.00103417" ixz="0.80199628" iyy="6.08689388" iyz="0.00105311" izz="4.96191932"/>

Commit message: Optical frame and mesh for gazebo cameras

File: sawyer_description/urdf/sawyer_base.gazebo.xacro (robot description, xacro)
@@ -54,10 +54,14 @@
     <provideFeedback>true</provideFeedback>
   </gazebo>
-  <!-- Gazebo-Specific Sensor Properties -->
-  <gazebo reference="head_camera">
+   <joint name="head_camera_optical_joint" type="fixed">
+    <origin xyz="0 0 0" rpy="${-pi} ${-pi/2.0} ${-pi/2.0}"/>
+    <parent link="head_camera"/>
+    <child link="head_camera_optical"/>
+  </joint>
+  <link name="head_camera_optical"/>
+  <gazebo reference="head_camera_optical">
     <sensor name="head_camera" type="camera">
       <update_rate>6.75</update_rate>
       <camera name="head_camera">
-        <pose>-1.570796 -1.570796 0.0 0.0 0.0 0.0</pose>
         <horizontal_fov>2.00787026</horizontal_fov>
         <distortion>
@@ -96,13 +100,17 @@
         <focalLength>407.391526</focalLength>
       </plugin>
-<visualize>true</visualize>
     </sensor>
   </gazebo>
-  <gazebo reference="right_hand_camera">
+  <joint name="right_hand_camera_optical_joint" type="fixed">
+    <origin xyz="0 0 0" rpy="${-pi} ${-pi/2.0} ${-pi/2.0}"/>
+    <parent link="right_hand_camera"/>
+    <child link="right_hand_camera_optical"/>
+  </joint>
+  <link name="right_hand_camera_optical"/>
+  <gazebo reference="right_hand_camera_optical">
     <sensor name="right_hand_camera" type="camera">
       <update_rate>5.0</update_rate>
       <camera name="right_hand_camera">
-        <pose>0.0 0.0 0.0 0.0 0.0 0.0 </pose>
-        <horizontal_fov>1.0992892</horizontal_fov>
+        <!-- horizontal_fov>1.0992892</horizontal_fov -->
         <image>
           <width>752</width>
@@ -114,12 +122,4 @@
           <far>300</far>
         </clip>
-        <distortion>
-          <k1>-0.442</k1>
-          <k2>0.273</k2>
-          <k3>-0.123</k3>
-          <p1>0.0</p1>
-          <p2>0.0</p2>
-          <center>365.734985 237.988998</center>
-        </distortion>
       </camera>
       <plugin filename="libgazebo_ros_camera.so" name="camera_controller">
@@ -130,15 +130,5 @@
         <cameraInfoTopicName>/io/internal_camera/right_hand_camera/camera_info</cameraInfoTopicName>
         <frameName>right_hand_camera</frameName>
-        <hackBaseline>0.0</hackBaseline>
-        <distortionK1>-0.442</distortionK1>
-        <distortionK2>0.273</distortionK2>
-        <distortionK3>-0.123</distortionK3>
-        <distortionT1>0.0</distortionT1>
-        <distortionT2>0.0</distortionT2>
-        <Cx>365.734985</Cx>
-        <Cy>237.988998</Cy>
-        <focalLength>613.760435</focalLength>
       </plugin>
-<visualize>true</visualize>
     </sensor>
   </gazebo>

Commit message: First pass at cognex light strobe

File: sawyer_description/urdf/sawyer_base.gazebo.xacro (robot description, xacro)
@@ -110,5 +110,34 @@
     <child link="right_hand_camera_optical"/>
   </joint>
-  <link name="right_hand_camera_optical"/>
+  <link name="right_hand_camera_optical">
+    <!-- light name="cognex_strobe" type="spot">
+      <cast_shadows>true</cast_shadows>
+      <pose>0 0 0.1 0 0 0</pose -->
+      <!-- diffuse>126 126 126 255</diffuse -->
+      <!-- specular>23 23 23 255</specular -->
+      <!-- diffuse>0.5 0.5 0.5 1.0</diffuse>
+      <specular>0.1 0.1 0.1 1.0</specular>
+      <attenuation>
+        <range>2</range>
+        <linear>0.01</linear>
+        <constant>0.12</constant>
+        <quadratic>0.00</quadratic>
+      </attenuation>
+      <spot>
+        <inner_angle>0.6</inner_angle>
+        <outer_angle>0.6</outer_angle>
+        <falloff>1.5</falloff>
+      </spot>
+    </light -->
+  </link>
+  <plugin name="attach_light" filename="libAttachLightPlugin.so">
+    <link>
+      <link_name>right_hand_camera_optical</link_name>
+      <light>
+        <pose>0 0 0.1 0 0 0</pose>
+        <light_name>spot</light_name>
+      </light>
+    </link>
+  </plugin>
   <gazebo reference="right_hand_camera_optical">
     <sensor name="right_hand_camera" type="camera">
