Commit message: Added gazebo xacro tag pass-through

File: sawyer_description/urdf/sawyer.urdf.xacro (robot description, xacro)
@@ -9,5 +9,7 @@
   <!-- Electric Gripper End Effector -->
   <xacro:if value="$(arg electric_gripper)">
-    <xacro:include filename="$(find sawyer_description)/urdf/sawyer_electric_gripper.urdf.xacro"/>
+    <xacro:include filename="$(find sawyer_description)/urdf/sawyer_electric_gripper.urdf.xacro">
+      <xacro:arg name="gazebo" value="${gazebo}"/>
+    </xacro:include>
   </xacro:if>
 </robot>

File: sawyer_description/urdf/sawyer_electric_gripper.urdf.xacro (robot description, xacro)
@@ -1,6 +1,14 @@
 <?xml version="1.0" ?>
 <robot name="end_effector" xmlns:xacro="http://www.ros.org/wiki/xacro">
+  <xacro:arg name="gazebo" default="false"/>
+  <xacro:if value="$(arg gazebo)">
+    <xacro:property name="gazebo_tag" value="true" scope="local"/>
+  </xacro:if>
+  <xacro:unless value="$(arg gazebo)">
+    <xacro:property name="gazebo_tag" value="false" scope="local"/>
+  </xacro:unless>
   <xacro:include filename="$(find intera_tools_description)/urdf/electric_gripper/rethink_electric_gripper.xacro" />
   <xacro:rethink_electric_gripper side="right"
+                                  gazebo="${gazebo_tag}"
                                   use_connector_plate="true"
                                   l_finger="standard_narrow"

Commit message: Update URDF, Xacro Args, & Sim Dynamics params
New URDF Xacro args:
- Adds "static" parameter for linking Sawyer to world frame in Gazebo
- Adds "pedestal" parameter for removing Sawyer's pedestal and
  associated frames
- Removed minimum inertia macro as it is no longer needed
- Made the <dynamics> tag values lower in accordance with tuned gains

File: sawyer_description/urdf/sawyer.urdf.xacro (robot description, xacro)
@@ -2,14 +2,23 @@
 <robot name="sawyer" xmlns:xacro="http://www.ros.org/wiki/xacro">
   <xacro:arg name="gazebo" default="false"/>
+  <xacro:arg name="pedestal" default="true"/>
+  <xacro:arg name="static" default="true"/>
   <xacro:arg name="electric_gripper" default="false"/>
   <!-- Sawyer Base URDF -->
   <xacro:include filename="$(find sawyer_description)/urdf/sawyer_base.urdf.xacro">
     <xacro:arg name="gazebo" value="${gazebo}"/>
+    <xacro:arg name="pedestal" value="${pedestal}"/>
   </xacro:include>
+  <xacro:if value="$(arg gazebo)">
+  <xacro:include filename="$(find sawyer_description)/urdf/sawyer_base.gazebo.xacro">
+    <xacro:arg name="static" value="${static}"/>
+    <xacro:arg name="pedestal" value="${pedestal}"/>
+  </xacro:include>
+  </xacro:if>
   <!-- Electric Gripper End Effector -->
   <xacro:if value="$(arg electric_gripper)">
-    <xacro:include filename="$(find sawyer_description)/urdf/sawyer_electric_gripper.urdf.xacro">
-      <xacro:arg name="gazebo" value="${gazebo}"/>
-    </xacro:include>
+  <xacro:include filename="$(find sawyer_description)/urdf/sawyer_electric_gripper.urdf.xacro">
+    <xacro:arg name="gazebo" value="${gazebo}"/>
+  </xacro:include>
   </xacro:if>
 </robot>

File: sawyer_description/urdf/sawyer_base.gazebo.xacro (robot description, xacro)
@@ -1,4 +1,6 @@
 <?xml version="1.0" ?>
 <robot name="baxter" xmlns:xacro="http://www.ros.org/wiki/xacro">
+  <xacro:arg name="pedestal" default="true"/>
+  <xacro:arg name="static" default="true"/>
   <!-- ros_control plugin -->
   <gazebo>
@@ -11,12 +13,16 @@
   </gazebo>
   <!-- Gazebo-Specific Link Properties -->
+<xacro:if value="$(arg static)">
   <link name="world"/>
-    <joint name="fixed" type="fixed">
+  <joint name="fixed" type="fixed">
       <parent link="world"/>
       <child link="base"/>
   </joint>
+</xacro:if>
+<xacro:if value="$(arg pedestal)">
   <gazebo reference="pedestal">
     <material>Gazebo/FlatBlack</material>
   </gazebo>
+</xacro:if>
   <gazebo reference="torso">
     <self_collide>true</self_collide>

File: sawyer_description/urdf/sawyer_base.urdf.xacro (robot description, xacro)
@@ -2,17 +2,5 @@
 <robot name="sawyer" xmlns:xacro="http://www.ros.org/wiki/xacro">
   <xacro:arg name="gazebo" default="false"/>
-  <xacro:if value="$(arg gazebo)">
-    <!-- Gazebo Tags -->
-    <xacro:include filename="$(find sawyer_description)/urdf/sawyer_base.gazebo.xacro" />
-  </xacro:if>
-  <xacro:macro name="gazebo_minimum_inertia">
-  <!--  In Gazebo, links with zero principal moment of inertia (ixx, iyy, izz) could lead to infinite acceleration under any finite torque application.
-      http://gazebosim.org/tutorials/?tut=ros_urdf -->
-    <inertial>
-      <origin rpy="0 0 0" xyz="0 0 0"/>
-      <mass value="0.01"/>
-      <inertia ixx="0.01" ixy="0" ixz="0" iyy="0.01" iyz="0" izz="0.01"/>
-    </inertial>
-  </xacro:macro>
+  <xacro:arg name="pedestal" default="true"/>
   <material name="black">
     <color rgba="0 0 0 1"/>
@@ -30,9 +18,5 @@
     <color rgba="0.75294 0.75294 0.75294 1"/>
   </material>
-  <link name="base">
-<xacro:if value="$(arg gazebo)">
-    <xacro:gazebo_minimum_inertia />
-</xacro:if>
-  </link>
+  <link name="base"/>
   <link name="torso">
     <visual>
@@ -45,7 +29,4 @@
       </material>
     </visual>
-<xacro:if value="$(arg gazebo)">
-    <xacro:gazebo_minimum_inertia />
-</xacro:if>
 <xacro:unless value="$(arg gazebo)">
     <inertial>
@@ -56,4 +37,5 @@
 </xacro:unless>
   </link>
+<xacro:if value="$(arg pedestal)">
   <link name="pedestal">
     <visual>
@@ -83,7 +65,4 @@
       </geometry>
     </collision>
-<xacro:if value="$(arg gazebo)">
-    <xacro:gazebo_minimum_inertia />
-</xacro:if>
   </link>
   <joint name="controller_box_fixed" type="fixed">
@@ -99,7 +78,4 @@
       </geometry>
     </collision>
-<xacro:if value="$(arg gazebo)">
-    <xacro:gazebo_minimum_inertia />
-</xacro:if>
   </link>
   <joint name="pedestal_feet_fixed" type="fixed">
@@ -108,4 +84,15 @@
     <child link="pedestal_feet"/>
   </joint>
+  <joint name="pedestal_fixed" type="fixed">
+    <origin rpy="0 0 0" xyz="0.0 0.0 0.0"/>
+    <parent link="base"/>
+    <child link="pedestal"/>
+  </joint>
+</xacro:if>
+  <joint name="right_arm_mount" type="fixed">
+    <origin rpy="0 0 0" xyz="0.0 0.0 0.0"/>
+    <parent link="base"/>
+    <child link="right_arm_base_link"/>
+  </joint>
   <joint name="torso_t0" type="fixed">
     <origin rpy="0 0 0" xyz="0 0 0"/>
@@ -113,14 +100,4 @@
     <child link="torso"/>
   </joint>
-  <joint name="pedestal_fixed" type="fixed">
-    <origin rpy="0 0 0" xyz="0.0 0.0 0.0"/>
-    <parent link="base"/>
-    <child link="pedestal"/>
-  </joint>
-  <joint name="right_arm_mount" type="fixed">
-    <origin rpy="0 0 0" xyz="0.0 0.0 0.0"/>
-    <parent link="base"/>
-    <child link="right_arm_base_link"/>
-  </joint>
   <link name="right_arm_base_link">
     <inertial>
@@ -170,5 +147,5 @@
     <limit effort="80.0" lower="-3.0503" upper="3.0503" velocity="1.74"/>
 <xacro:if value="$(arg gazebo)">
-    <dynamics damping="15.0" friction="5.0"/>
+    <dynamics damping="5.0" friction="2.0"/>
 </xacro:if>
   </joint>
@@ -204,7 +181,4 @@
   </joint>
   <link name="right_torso_itb">
-<xacro:if value="$(arg gazebo)">
-    <xacro:gazebo_minimum_inertia />
-</xacro:if>
 <xacro:unless value="$(arg gazebo)">
     <inertial>
@@ -308,5 +282,5 @@
     <limit effort="40.0" lower="-3.0439" upper="3.0439" velocity="1.957"/>
  <xacro:if value="$(arg gazebo)">
-    <dynamics damping="15.0" friction="5.0"/>
+    <dynamics damping="1.0" friction="0.5"/>
 </xacro:if>
   </joint>
@@ -338,11 +312,8 @@
     <limit effort="9.0" lower="-2.9761" upper="2.9761" velocity="3.485"/>
 <xacro:if value="$(arg gazebo)">
-    <dynamics damping="6.0" friction="1.0"/>
+    <dynamics damping="2.0" friction="1.0"/>
 </xacro:if>
   </joint>
   <link name="right_arm_itb">
-<xacro:if value="$(arg gazebo)">
-    <xacro:gazebo_minimum_inertia />
-</xacro:if>
 <xacro:unless value="$(arg gazebo)">
     <inertial>
@@ -386,12 +357,8 @@
     <limit effort="9.0" lower="-2.9761" upper="2.9761" velocity="3.485"/>
 <xacro:if value="$(arg gazebo)">
-    <dynamics damping="5.5" friction="1.2"/>
-</xacro:if>
-  </joint>
-  <link name="right_hand_camera">
-<xacro:if value="$(arg gazebo)">
-    <xacro:gazebo_minimum_inertia />
-</xacro:if>
-  </link>
+    <dynamics damping="1.0" friction="0.5"/>
+</xacro:if>
+  </joint>
+  <link name="right_hand_camera"/>
   <joint name="right_hand_camera" type="fixed">
     <origin rpy="0 1.57079632679 0" xyz="0.039552 -0.033 0.0695"/>
@@ -400,9 +367,5 @@
     <axis xyz="0 0 0"/>
   </joint>
-  <link name="right_wrist">
-<xacro:if value="$(arg gazebo)">
-    <xacro:gazebo_minimum_inertia />
-</xacro:if>
-  </link>
+  <link name="right_wrist"/>
   <joint name="right_wrist" type="fixed">
     <origin rpy="1.57079632679 0 0" xyz="0 0 0.10541"/>
@@ -452,5 +415,9 @@
     </collision>
 <xacro:if value="$(arg gazebo)">
-      <xacro:gazebo_minimum_inertia />
+    <inertial>
+      <origin rpy="0 0 0" xyz="0 0.1 0"/>
+      <mass value="0.01"/>
+      <inertia ixx="0.01" ixy="0.01" ixz="0.01" iyy="0.01" iyz="0.01" izz="0.01"/>
+  </inertial>
 </xacro:if>
 <xacro:unless value="$(arg gazebo)">
@@ -469,7 +436,4 @@
   </joint>
   <link name="right_l1_2">
-<xacro:if value="$(arg gazebo)">
-    <xacro:gazebo_minimum_inertia />
-</xacro:if>
 <xacro:unless value="$(arg gazebo)">
     <inertial>
@@ -493,7 +457,4 @@
   </joint>
   <link name="right_l2_2">
-<xacro:if value="$(arg gazebo)">
-    <xacro:gazebo_minimum_inertia />
-</xacro:if>
 <xacro:unless value="$(arg gazebo)">
     <inertial>
@@ -517,7 +478,4 @@
   </joint>
   <link name="right_l4_2">
-<xacro:if value="$(arg gazebo)">
-    <xacro:gazebo_minimum_inertia />
-</xacro:if>
 <xacro:unless value="$(arg gazebo)">
     <inertial>
@@ -554,7 +512,4 @@
       </geometry>
     </collision>
-<xacro:if value="$(arg gazebo)">
-    <xacro:gazebo_minimum_inertia />
-</xacro:if>
 <xacro:unless value="$(arg gazebo)">
     <inertial>
@@ -570,9 +525,5 @@
     <child link="screen"/>
   </joint>
-  <link name="head_camera">
-<xacro:if value="$(arg gazebo)">
-    <xacro:gazebo_minimum_inertia />
-</xacro:if>
-  </link>
+  <link name="head_camera"/>
   <joint name="head_camera" type="fixed">
     <origin rpy="-2.1293 0 -1.57079632679" xyz="0.0228027 0 0.216572"/>
