Commit message: Updated URDF for Xacro and gazebo

File: sawyer_description/urdf/sawyer_base.urdf.xacro (robot description, xacro)
@@ -1,8 +1,9 @@
 <?xml version="1.0" ?>
-<!-- =================================================================================== -->
-<!-- |    This document was autogenerated by xacro from ./urdf.xacro                   | -->
-<!-- |    EDITING THIS FILE BY HAND IS NOT RECOMMENDED                                 | -->
-<!-- =================================================================================== -->
 <robot name="sawyer" xmlns:xacro="http://www.ros.org/wiki/xacro">
+  <xacro:arg name="gazebo" default="false"/>
+  <xacro:if value="$(arg gazebo)">
+    <!-- Gazebo Tags -->
+    <xacro:include filename="$(find sawyer_description)/urdf/sawyer_base.gazebo.xacro" />
+  </xacro:if>
   <material name="black">
     <color rgba="0 0 0 1"/>
@@ -25,5 +26,5 @@
       <origin rpy="0 0 0" xyz="0 0 0"/>
       <geometry>
-        <box size="0 0 0"/>
+        <box size="0.001 0.001 0.001"/>
       </geometry>
       <material name="darkgray">

Commit message: Adds initial URDF damping and frict vals for sim

File: sawyer_description/urdf/sawyer_base.urdf.xacro (robot description, xacro)
@@ -145,4 +145,5 @@
     <axis xyz="0 0 1"/>
     <limit effort="80.0" lower="-3.0503" upper="3.0503" velocity="1.74"/>
+    <dynamics damping="5.0" friction="5.0"/>
   </joint>
   <link name="head">
@@ -172,4 +173,5 @@
     <axis xyz="0 0 1"/>
     <limit effort="8" lower="-5.0952" upper="0.9064" velocity="1.8"/>
+    <dynamics damping="1.0" friction="0.5"/>
   </joint>
   <link name="right_torso_itb">
@@ -212,4 +214,5 @@
     <axis xyz="0 0 1"/>
     <limit effort="80.0" lower="-3.8095" upper="2.2736" velocity="1.328"/>
+    <dynamics damping="5.0" friction="5.0"/>
   </joint>
   <link name="right_l2">
@@ -239,4 +242,5 @@
     <axis xyz="0 0 1"/>
     <limit effort="40.0" lower="-3.0426" upper="3.0426" velocity="1.957"/>
+    <dynamics damping="5.0" friction="5.0"/>
   </joint>
   <link name="right_l3">
@@ -266,4 +270,5 @@
     <axis xyz="0 0 1"/>
     <limit effort="40.0" lower="-3.0439" upper="3.0439" velocity="1.957"/>
+    <dynamics damping="5.0" friction="5.0"/>
   </joint>
   <link name="right_l4">
@@ -293,4 +298,5 @@
     <axis xyz="0 0 1"/>
     <limit effort="9.0" lower="-2.9761" upper="2.9761" velocity="3.485"/>
+    <dynamics damping="5.0" friction="5.0"/>
   </joint>
   <link name="right_arm_itb">
@@ -333,4 +339,5 @@
     <axis xyz="0 0 1"/>
     <limit effort="9.0" lower="-2.9761" upper="2.9761" velocity="3.485"/>
+    <dynamics damping="5.0" friction="5.0"/>
   </joint>
   <link name="right_hand_camera"/>
@@ -374,4 +381,5 @@
     <axis xyz="0 0 1"/>
     <limit effort="9.0" lower="-4.7124" upper="4.7124" velocity="4.545"/>
+    <dynamics damping="5.0" friction="5.0"/>
   </joint>
   <link name="right_hand">

Commit message: Lowered friction and damping on j4-j6 in URDF
Based on a conversation with the Controls team

File: sawyer_description/urdf/sawyer_base.urdf.xacro (robot description, xacro)
@@ -298,5 +298,5 @@
     <axis xyz="0 0 1"/>
     <limit effort="9.0" lower="-2.9761" upper="2.9761" velocity="3.485"/>
-    <dynamics damping="5.0" friction="5.0"/>
+    <dynamics damping="2.0" friction="2.0"/>
   </joint>
   <link name="right_arm_itb">
@@ -339,5 +339,5 @@
     <axis xyz="0 0 1"/>
     <limit effort="9.0" lower="-2.9761" upper="2.9761" velocity="3.485"/>
-    <dynamics damping="5.0" friction="5.0"/>
+    <dynamics damping="2.0" friction="2.0"/>
   </joint>
   <link name="right_hand_camera"/>
@@ -381,5 +381,5 @@
     <axis xyz="0 0 1"/>
     <limit effort="9.0" lower="-4.7124" upper="4.7124" velocity="4.545"/>
-    <dynamics damping="5.0" friction="5.0"/>
+    <dynamics damping="2.0" friction="2.0"/>
   </joint>
   <link name="right_hand">

Commit message: reduce movement

File: sawyer_description/urdf/sawyer_base.urdf.xacro (robot description, xacro)
@@ -21,5 +21,11 @@
     <color rgba="0.75294 0.75294 0.75294 1"/>
   </material>
-  <link name="base"/>
+  <link name="base">
+      <inertial>
+        <origin rpy="0 0 0" xyz="0 0 0"/>
+        <mass value="0.01"/>
+        <inertia ixx="0.1" ixy="0" ixz="0" iyy="0.1" iyz="0" izz="0.1"/>
+      </inertial>
+  </link>
   <link name="torso">
     <visual>
@@ -34,6 +40,6 @@
     <inertial>
       <origin rpy="0 0 0" xyz="0.000000 0.000000 0.000000"/>
-      <mass value="0.0001"/>
-      <inertia ixx="1e-08" ixy="0" ixz="0" iyy="1e-08" iyz="0" izz="1e-08"/>
+      <mass value="0.01"/>
+      <inertia ixx="0.1" ixy="0" ixz="0" iyy="0.1" iyz="0" izz="0.1"/>
     </inertial>
   </link>
@@ -65,4 +71,9 @@
       </geometry>
     </collision>
+    <inertial>
+      <origin rpy="0 0 0" xyz="0 0 0"/>
+      <mass value="0.01"/>
+      <inertia ixx="0.1" ixy="0" ixz="0" iyy="0.1" iyz="0" izz="0.1"/>
+    </inertial>
   </link>
   <joint name="controller_box_fixed" type="fixed">
@@ -78,4 +89,9 @@
       </geometry>
     </collision>
+    <inertial>
+      <origin rpy="0 0 0" xyz="0 0 0"/>
+      <mass value="0.01"/>
+      <inertia ixx="0.1" ixy="0" ixz="0" iyy="0.1" iyz="0" izz="0.1"/>
+    </inertial>
   </link>
   <joint name="pedestal_feet_fixed" type="fixed">
@@ -175,17 +191,4 @@
     <dynamics damping="1.0" friction="0.5"/>
   </joint>
-  <link name="right_torso_itb">
-    <inertial>
-      <origin rpy="0 0 0" xyz="0.000000 0.000000 0.000000"/>
-      <mass value="0.0001"/>
-      <inertia ixx="1e-08" ixy="0" ixz="0" iyy="1e-08" iyz="0" izz="1e-08"/>
-    </inertial>
-  </link>
-  <joint name="right_torso_itb" type="fixed">
-    <origin rpy="0 -1.57079632679 0" xyz="-.055 0 .22"/>
-    <parent link="right_l0"/>
-    <child link="right_torso_itb"/>
-    <axis xyz="0 0 1"/>
-  </joint>
   <link name="right_l1">
     <inertial>
@@ -300,17 +303,4 @@
     <dynamics damping="2.0" friction="2.0"/>
   </joint>
-  <link name="right_arm_itb">
-    <inertial>
-      <origin rpy="0 0 0" xyz="0.000000 0.000000 0.000000"/>
-      <mass value="0.0001"/>
-      <inertia ixx="1e-08" ixy="0" ixz="0" iyy="1e-08" iyz="0" izz="1e-08"/>
-    </inertial>
-  </link>
-  <joint name="right_arm_itb" type="fixed">
-    <origin rpy="0 -1.57079632679 0" xyz="-.055 0 .075"/>
-    <parent link="right_l4"/>
-    <child link="right_arm_itb"/>
-    <axis xyz="0 0 1"/>
-  </joint>
   <link name="right_l5">
     <inertial>
@@ -341,5 +331,11 @@
     <dynamics damping="2.0" friction="2.0"/>
   </joint>
-  <link name="right_hand_camera"/>
+  <link name="right_hand_camera">
+      <inertial>
+        <origin rpy="0 0 0" xyz="0 0 0"/>
+        <mass value="0.01"/>
+        <inertia ixx="0.1" ixy="0" ixz="0" iyy="0.1" iyz="0" izz="0.1"/>
+      </inertial>
+  </link>
   <joint name="right_hand_camera" type="fixed">
     <origin rpy="0 1.57079632679 0" xyz="0.039552 -0.033 0.0695"/>
@@ -348,5 +344,11 @@
     <axis xyz="0 0 0"/>
   </joint>
-  <link name="right_wrist"/>
+  <link name="right_wrist">
+      <inertial>
+        <origin rpy="0 0 0" xyz="0 0 0"/>
+        <mass value="0.01"/>
+        <inertia ixx="0.1" ixy="0" ixz="0" iyy="0.1" iyz="0" izz="0.1"/>
+      </inertial>
+  </link>
   <joint name="right_wrist" type="fixed">
     <origin rpy="1.57079632679 0 0" xyz="0 0 0.10541"/>
@@ -380,5 +382,6 @@
     <child link="right_l6"/>
     <axis xyz="0 0 1"/>
-    <limit effort="9.0" lower="-4.7124" upper="4.7124" velocity="4.545"/>
+    <!-- limit effort="9.0" lower="-4.7124" upper="4.7124" velocity="4.545"/ -->
+    <limit effort="9.0" lower="-3.14" upper="3.14" velocity="4.545"/>
     <dynamics damping="2.0" friction="2.0"/>
   </joint>
@@ -391,7 +394,7 @@
     </collision>
     <inertial>
-      <origin rpy="0 0 0" xyz="1.0E-08 1.0E-08 1.0E-08"/>
-      <mass value="1.0E-08"/>
-      <inertia ixx="1.0E-08" ixy="1.0E-08" ixz="1.0E-08" iyy="1.0E-08" iyz="1.0E-08" izz="1.0E-08"/>
+      <origin rpy="0 0 0" xyz="0 0 0"/>
+      <mass value="0.01"/>
+      <inertia ixx="0.1" ixy="0" ixz="0" iyy="0.1" iyz="0" izz="0.1"/>
     </inertial>
   </link>
@@ -401,62 +404,5 @@
     <parent link="right_l6"/>
     <child link="right_hand"/>
-  </joint>
-  <link name="right_l1_2">
-    <inertial>
-      <origin rpy="0 0 0" xyz="1.0E-08 1.0E-08 1.0E-08"/>
-      <mass value="1.0E-08"/>
-      <inertia ixx="1.0E-08" ixy="1.0E-08" ixz="1.0E-08" iyy="1.0E-08" iyz="1.0E-08" izz="1.0E-08"/>
-    </inertial>
-    <collision>
-      <origin rpy="0 0 0" xyz="0 0 0.035"/>
-      <geometry>
-        <cylinder length="0.14" radius="0.07"/>
-      </geometry>
-    </collision>
-  </link>
-  <joint name="right_j1_2" type="fixed">
-    <origin rpy="0 0 0" xyz="0 0 0"/>
-    <parent link="right_l1"/>
-    <child link="right_l1_2"/>
-    <axis xyz="0 0 1"/>
-  </joint>
-  <link name="right_l2_2">
-    <inertial>
-      <origin rpy="0 0 0" xyz="1.0E-08 1.0E-08 1.0E-08"/>
-      <mass value="1.0E-08"/>
-      <inertia ixx="1.0E-08" ixy="1.0E-08" ixz="1.0E-08" iyy="1.0E-08" iyz="1.0E-08" izz="1.0E-08"/>
-    </inertial>
-    <collision>
-      <origin rpy="0 0 0" xyz="0 0 0.26"/>
-      <geometry>
-        <sphere radius="0.06"/>
-      </geometry>
-    </collision>
-  </link>
-  <joint name="right_j2_2" type="fixed">
-    <origin rpy="0 0 0" xyz="0 0 0"/>
-    <parent link="right_l2"/>
-    <child link="right_l2_2"/>
-    <axis xyz="0 0 1"/>
-  </joint>
-  <link name="right_l4_2">
-    <inertial>
-      <origin rpy="0 0 0" xyz="1.0E-08 1.0E-08 1.0E-08"/>
-      <mass value="1.0E-08"/>
-      <inertia ixx="1.0E-08" ixy="1.0E-08" ixz="1.0E-08" iyy="1.0E-08" iyz="1.0E-08" izz="1.0E-08"/>
-    </inertial>
-    <collision>
-      <origin rpy="0 0 0" xyz="0 0.01 0.26"/>
-      <geometry>
-        <sphere radius="0.06"/>
-      </geometry>
-    </collision>
-  </link>
-  <joint name="right_j4_2" type="fixed">
-    <origin rpy="0 0 0" xyz="0 0 0"/>
-    <parent link="right_l4"/>
-    <child link="right_l4_2"/>
-    <axis xyz="0 0 1"/>
-  </joint>
+</joint>
   <link name="screen">
     <visual>
@@ -475,6 +421,6 @@
     <inertial>
       <origin rpy="0 0 0" xyz="0 0 0"/>
-      <mass value="0.0001"/>
-      <inertia ixx="1e-08" ixy="0" ixz="0" iyy="1e-08" iyz="0" izz="1e-08"/>
+      <mass value="0.01"/>
+      <inertia ixx="0.1" ixy="0" ixz="0" iyy="0.1" iyz="0" izz="0.1"/>
     </inertial>
   </link>
@@ -484,5 +430,11 @@
     <child link="screen"/>
   </joint>
-  <link name="head_camera"/>
+  <link name="head_camera">
+      <inertial>
+        <origin rpy="0 0 0" xyz="0 0 0"/>
+        <mass value="0.01"/>
+        <inertia ixx="0.1" ixy="0" ixz="0" iyy="0.1" iyz="0" izz="0.1"/>
+      </inertial>
+  </link>
   <joint name="head_camera" type="fixed">
     <origin rpy="-2.1293 0 -1.57079632679" xyz="0.0228027 0 0.216572"/>

Commit message: Sim Controller Tuning
Corresponds with RethinkRobotics/sawyer_simulator#35

Now that all the controllers have been created, and the software
processes are in place to emulate the real Sawyer robot's API's, this is
the latest round of tuning for Sawyer's Position(&Trajectory) and
Velocity Controllers. This corresponds with some URDF tweaks in order to
make Gazebo happy: increased zero mass & inertia links to have a minimum
mass and inertia, and re-tuned joint damping and friction for
simulation.

This was tested with a computer capable of running Sawyer in Gazebo at a
consistent Real Time Factor of 1.0 throughout the duration of testing.

    Trajectory Mode works well(-ish) with MoveIt! Nearly all
trajectories execute without violating the real Sawyer's joint tracking
or Goal Velocity constraints
    Regular Position Mode moves at nearly the same speed as the real
Sawyer
    Velocity Mode works well with the joint_velocity_wobbler.py example
script

The one slight downside is that with the retuning, and mass/inertia
tweaks, Gravity Compensation is just barely not enough to hold up the
arm when commanding only Zero Torques. Funny enough, this is actually
closer to the reality of the real Sawyer.

File: sawyer_description/urdf/sawyer_base.urdf.xacro (robot description, xacro)
@@ -6,4 +6,13 @@
     <xacro:include filename="$(find sawyer_description)/urdf/sawyer_base.gazebo.xacro" />
   </xacro:if>
+  <xacro:macro name="gazebo_minimum_inertia">
+  <!--  In Gazebo, links with zero principal moment of inertia (ixx, iyy, izz) could lead to infinite acceleration under any finite torque application.
+      http://gazebosim.org/tutorials/?tut=ros_urdf -->
+    <inertial>
+      <origin rpy="0 0 0" xyz="0 0 0"/>
+      <mass value="0.01"/>
+      <inertia ixx="0.01" ixy="0" ixz="0" iyy="0.01" iyz="0" izz="0.01"/>
+    </inertial>
+  </xacro:macro>
   <material name="black">
     <color rgba="0 0 0 1"/>
@@ -21,5 +30,9 @@
     <color rgba="0.75294 0.75294 0.75294 1"/>
   </material>
-  <link name="base"/>
+  <link name="base">
+<xacro:if value="$(arg gazebo)">
+    <xacro:gazebo_minimum_inertia />
+</xacro:if>
+  </link>
   <link name="torso">
     <visual>
@@ -32,4 +45,8 @@
       </material>
     </visual>
+<xacro:if value="$(arg gazebo)">
+    <xacro:gazebo_minimum_inertia />
+</xacro:if>
+<xacro:unless value="$(arg gazebo)">
     <inertial>
       <origin rpy="0 0 0" xyz="0.000000 0.000000 0.000000"/>
@@ -37,4 +54,5 @@
       <inertia ixx="1e-08" ixy="0" ixz="0" iyy="1e-08" iyz="0" izz="1e-08"/>
     </inertial>
+</xacro:unless>
   </link>
   <link name="pedestal">
@@ -65,4 +83,7 @@
       </geometry>
     </collision>
+<xacro:if value="$(arg gazebo)">
+    <xacro:gazebo_minimum_inertia />
+</xacro:if>
   </link>
   <joint name="controller_box_fixed" type="fixed">
@@ -78,4 +99,7 @@
       </geometry>
     </collision>
+<xacro:if value="$(arg gazebo)">
+    <xacro:gazebo_minimum_inertia />
+</xacro:if>
   </link>
   <joint name="pedestal_feet_fixed" type="fixed">
@@ -145,5 +169,7 @@
     <axis xyz="0 0 1"/>
     <limit effort="80.0" lower="-3.0503" upper="3.0503" velocity="1.74"/>
-    <dynamics damping="5.0" friction="5.0"/>
+<xacro:if value="$(arg gazebo)">
+    <dynamics damping="15.0" friction="5.0"/>
+</xacro:if>
   </joint>
   <link name="head">
@@ -173,7 +199,13 @@
     <axis xyz="0 0 1"/>
     <limit effort="8" lower="-5.0952" upper="0.9064" velocity="1.8"/>
+<xacro:if value="$(arg gazebo)">
     <dynamics damping="1.0" friction="0.5"/>
+</xacro:if>
   </joint>
   <link name="right_torso_itb">
+<xacro:if value="$(arg gazebo)">
+    <xacro:gazebo_minimum_inertia />
+</xacro:if>
+<xacro:unless value="$(arg gazebo)">
     <inertial>
       <origin rpy="0 0 0" xyz="0.000000 0.000000 0.000000"/>
@@ -181,4 +213,5 @@
       <inertia ixx="1e-08" ixy="0" ixz="0" iyy="1e-08" iyz="0" izz="1e-08"/>
     </inertial>
+</xacro:unless>
   </link>
   <joint name="right_torso_itb" type="fixed">
@@ -214,5 +247,7 @@
     <axis xyz="0 0 1"/>
     <limit effort="80.0" lower="-3.8095" upper="2.2736" velocity="1.328"/>
-    <dynamics damping="5.0" friction="5.0"/>
+<xacro:if value="$(arg gazebo)">
+    <dynamics damping="5.0" friction="2.0"/>
+</xacro:if>
   </joint>
   <link name="right_l2">
@@ -242,5 +277,7 @@
     <axis xyz="0 0 1"/>
     <limit effort="40.0" lower="-3.0426" upper="3.0426" velocity="1.957"/>
-    <dynamics damping="5.0" friction="5.0"/>
+<xacro:if value="$(arg gazebo)">
+    <dynamics damping="5.0" friction="2.0"/>
+</xacro:if>
   </joint>
   <link name="right_l3">
@@ -270,5 +307,7 @@
     <axis xyz="0 0 1"/>
     <limit effort="40.0" lower="-3.0439" upper="3.0439" velocity="1.957"/>
-    <dynamics damping="5.0" friction="5.0"/>
+ <xacro:if value="$(arg gazebo)">
+    <dynamics damping="15.0" friction="5.0"/>
+</xacro:if>
   </joint>
   <link name="right_l4">
@@ -298,7 +337,13 @@
     <axis xyz="0 0 1"/>
     <limit effort="9.0" lower="-2.9761" upper="2.9761" velocity="3.485"/>
-    <dynamics damping="2.0" friction="2.0"/>
+<xacro:if value="$(arg gazebo)">
+    <dynamics damping="6.0" friction="1.0"/>
+</xacro:if>
   </joint>
   <link name="right_arm_itb">
+<xacro:if value="$(arg gazebo)">
+    <xacro:gazebo_minimum_inertia />
+</xacro:if>
+<xacro:unless value="$(arg gazebo)">
     <inertial>
       <origin rpy="0 0 0" xyz="0.000000 0.000000 0.000000"/>
@@ -306,4 +351,5 @@
       <inertia ixx="1e-08" ixy="0" ixz="0" iyy="1e-08" iyz="0" izz="1e-08"/>
     </inertial>
+</xacro:unless>
   </link>
   <joint name="right_arm_itb" type="fixed">
@@ -339,7 +385,13 @@
     <axis xyz="0 0 1"/>
     <limit effort="9.0" lower="-2.9761" upper="2.9761" velocity="3.485"/>
-    <dynamics damping="2.0" friction="2.0"/>
-  </joint>
-  <link name="right_hand_camera"/>
+<xacro:if value="$(arg gazebo)">
+    <dynamics damping="5.5" friction="1.2"/>
+</xacro:if>
+  </joint>
+  <link name="right_hand_camera">
+<xacro:if value="$(arg gazebo)">
+    <xacro:gazebo_minimum_inertia />
+</xacro:if>
+  </link>
   <joint name="right_hand_camera" type="fixed">
     <origin rpy="0 1.57079632679 0" xyz="0.039552 -0.033 0.0695"/>
@@ -348,5 +400,9 @@
     <axis xyz="0 0 0"/>
   </joint>
-  <link name="right_wrist"/>
+  <link name="right_wrist">
+<xacro:if value="$(arg gazebo)">
+    <xacro:gazebo_minimum_inertia />
+</xacro:if>
+  </link>
   <joint name="right_wrist" type="fixed">
     <origin rpy="1.57079632679 0 0" xyz="0 0 0.10541"/>
@@ -380,6 +436,11 @@
     <child link="right_l6"/>
     <axis xyz="0 0 1"/>
+<xacro:if value="$(arg gazebo)">
+    <limit effort="9.0" lower="-3.14" upper="3.14" velocity="4.545"/>
+    <dynamics damping="1.0" friction="0.5"/>
+</xacro:if>
+<xacro:unless value="$(arg gazebo)">
     <limit effort="9.0" lower="-4.7124" upper="4.7124" velocity="4.545"/>
-    <dynamics damping="2.0" friction="2.0"/>
+</xacro:unless>
   </joint>
   <link name="right_hand">
@@ -390,4 +451,8 @@
       </geometry>
     </collision>
+<xacro:if value="$(arg gazebo)">
+      <xacro:gazebo_minimum_inertia />
+</xacro:if>
+<xacro:unless value="$(arg gazebo)">
     <inertial>
       <origin rpy="0 0 0" xyz="1.0E-08 1.0E-08 1.0E-08"/>
@@ -395,4 +460,5 @@
       <inertia ixx="1.0E-08" ixy="1.0E-08" ixz="1.0E-08" iyy="1.0E-08" iyz="1.0E-08" izz="1.0E-08"/>
     </inertial>
+</xacro:unless>
   </link>
   <joint name="right_hand" type="fixed">
@@ -403,4 +469,8 @@
   </joint>
   <link name="right_l1_2">
+<xacro:if value="$(arg gazebo)">
+    <xacro:gazebo_minimum_inertia />
+</xacro:if>
+<xacro:unless value="$(arg gazebo)">
     <inertial>
       <origin rpy="0 0 0" xyz="1.0E-08 1.0E-08 1.0E-08"/>
@@ -408,4 +478,5 @@
       <inertia ixx="1.0E-08" ixy="1.0E-08" ixz="1.0E-08" iyy="1.0E-08" iyz="1.0E-08" izz="1.0E-08"/>
     </inertial>
+</xacro:unless>
     <collision>
       <origin rpy="0 0 0" xyz="0 0 0.035"/>
@@ -422,4 +493,8 @@
   </joint>
   <link name="right_l2_2">
+<xacro:if value="$(arg gazebo)">
+    <xacro:gazebo_minimum_inertia />
+</xacro:if>
+<xacro:unless value="$(arg gazebo)">
     <inertial>
       <origin rpy="0 0 0" xyz="1.0E-08 1.0E-08 1.0E-08"/>
@@ -427,4 +502,5 @@
       <inertia ixx="1.0E-08" ixy="1.0E-08" ixz="1.0E-08" iyy="1.0E-08" iyz="1.0E-08" izz="1.0E-08"/>
     </inertial>
+</xacro:unless>
     <collision>
       <origin rpy="0 0 0" xyz="0 0 0.26"/>
@@ -441,4 +517,8 @@
   </joint>
   <link name="right_l4_2">
+<xacro:if value="$(arg gazebo)">
+    <xacro:gazebo_minimum_inertia />
+</xacro:if>
+<xacro:unless value="$(arg gazebo)">
     <inertial>
       <origin rpy="0 0 0" xyz="1.0E-08 1.0E-08 1.0E-08"/>
@@ -446,4 +526,5 @@
       <inertia ixx="1.0E-08" ixy="1.0E-08" ixz="1.0E-08" iyy="1.0E-08" iyz="1.0E-08" izz="1.0E-08"/>
     </inertial>
+</xacro:unless>
     <collision>
       <origin rpy="0 0 0" xyz="0 0.01 0.26"/>
@@ -473,4 +554,8 @@
       </geometry>
     </collision>
+<xacro:if value="$(arg gazebo)">
+    <xacro:gazebo_minimum_inertia />
+</xacro:if>
+<xacro:unless value="$(arg gazebo)">
     <inertial>
       <origin rpy="0 0 0" xyz="0 0 0"/>
@@ -478,4 +563,5 @@
       <inertia ixx="1e-08" ixy="0" ixz="0" iyy="1e-08" iyz="0" izz="1e-08"/>
     </inertial>
+</xacro:unless>
   </link>
   <joint name="display_joint" type="fixed">
@@ -484,5 +570,9 @@
     <child link="screen"/>
   </joint>
-  <link name="head_camera"/>
+  <link name="head_camera">
+<xacro:if value="$(arg gazebo)">
+    <xacro:gazebo_minimum_inertia />
+</xacro:if>
+  </link>
   <joint name="head_camera" type="fixed">
     <origin rpy="-2.1293 0 -1.57079632679" xyz="0.0228027 0 0.216572"/>
