Commit message: inertial and damping tuning

File: sawyer_description/urdf/sawyer_base.urdf.xacro (robot description, xacro)
@@ -6,4 +6,13 @@
     <xacro:include filename="$(find sawyer_description)/urdf/sawyer_base.gazebo.xacro" />
   </xacro:if>
+  <xacro:macro name="gazebo_minimum_inertia">
+  <!--  In Gazebo, links with zero principal moment of inertia (ixx, iyy, izz) could lead to infinite acceleration under any finite torque application.
+      http://gazebosim.org/tutorials/?tut=ros_urdf -->
+    <inertial>
+      <origin rpy="0 0 0" xyz="0 0 0"/>
+      <mass value="0.01"/>
+      <inertia ixx="0.001" ixy="0" ixz="0" iyy="0.001" iyz="0" izz="0.001"/>
+    </inertial>
+  </xacro:macro>
   <material name="black">
     <color rgba="0 0 0 1"/>
@@ -22,9 +31,7 @@
   </material>
   <link name="base">
-      <inertial>
-        <origin rpy="0 0 0" xyz="0 0 0"/>
-        <mass value="0.01"/>
-        <inertia ixx="0.1" ixy="0" ixz="0" iyy="0.1" iyz="0" izz="0.1"/>
-      </inertial>
+<xacro:if value="$(arg gazebo)">
+    <xacro:gazebo_minimum_inertia />
+</xacro:if>
   </link>
   <link name="torso">
@@ -38,9 +45,14 @@
       </material>
     </visual>
+<xacro:if value="$(arg gazebo)">
+    <xacro:gazebo_minimum_inertia />
+</xacro:if>
+<xacro:unless value="$(arg gazebo)">
     <inertial>
       <origin rpy="0 0 0" xyz="0.000000 0.000000 0.000000"/>
-      <mass value="0.01"/>
-      <inertia ixx="0.1" ixy="0" ixz="0" iyy="0.1" iyz="0" izz="0.1"/>
-    </inertial>
+      <mass value="0.0001"/>
+      <inertia ixx="1e-08" ixy="0" ixz="0" iyy="1e-08" iyz="0" izz="1e-08"/>
+    </inertial>
+</xacro:unless>
   </link>
   <link name="pedestal">
@@ -71,9 +83,7 @@
       </geometry>
     </collision>
-    <inertial>
-      <origin rpy="0 0 0" xyz="0 0 0"/>
-      <mass value="0.01"/>
-      <inertia ixx="0.1" ixy="0" ixz="0" iyy="0.1" iyz="0" izz="0.1"/>
-    </inertial>
+<xacro:if value="$(arg gazebo)">
+    <xacro:gazebo_minimum_inertia />
+</xacro:if>
   </link>
   <joint name="controller_box_fixed" type="fixed">
@@ -89,9 +99,7 @@
       </geometry>
     </collision>
-    <inertial>
-      <origin rpy="0 0 0" xyz="0 0 0"/>
-      <mass value="0.01"/>
-      <inertia ixx="0.1" ixy="0" ixz="0" iyy="0.1" iyz="0" izz="0.1"/>
-    </inertial>
+<xacro:if value="$(arg gazebo)">
+    <xacro:gazebo_minimum_inertia />
+</xacro:if>
   </link>
   <joint name="pedestal_feet_fixed" type="fixed">
@@ -161,5 +169,7 @@
     <axis xyz="0 0 1"/>
     <limit effort="80.0" lower="-3.0503" upper="3.0503" velocity="1.74"/>
-    <dynamics damping="5.0" friction="5.0"/>
+<xacro:if value="$(arg gazebo)">
+    <dynamics damping="5.0" friction="2.0"/>
+</xacro:if>
   </joint>
   <link name="head">
@@ -189,5 +199,25 @@
     <axis xyz="0 0 1"/>
     <limit effort="8" lower="-5.0952" upper="0.9064" velocity="1.8"/>
+<xacro:if value="$(arg gazebo)">
     <dynamics damping="1.0" friction="0.5"/>
+</xacro:if>
+  </joint>
+  <link name="right_torso_itb">
+<xacro:if value="$(arg gazebo)">
+    <xacro:gazebo_minimum_inertia />
+</xacro:if>
+<xacro:unless value="$(arg gazebo)">
+    <inertial>
+      <origin rpy="0 0 0" xyz="0.000000 0.000000 0.000000"/>
+      <mass value="0.0001"/>
+      <inertia ixx="1e-08" ixy="0" ixz="0" iyy="1e-08" iyz="0" izz="1e-08"/>
+    </inertial>
+</xacro:unless>
+  </link>
+  <joint name="right_torso_itb" type="fixed">
+    <origin rpy="0 -1.57079632679 0" xyz="-.055 0 .22"/>
+    <parent link="right_l0"/>
+    <child link="right_torso_itb"/>
+    <axis xyz="0 0 1"/>
   </joint>
   <link name="right_l1">
@@ -217,5 +247,7 @@
     <axis xyz="0 0 1"/>
     <limit effort="80.0" lower="-3.8095" upper="2.2736" velocity="1.328"/>
-    <dynamics damping="5.0" friction="5.0"/>
+<xacro:if value="$(arg gazebo)">
+    <dynamics damping="5.0" friction="2.0"/>
+</xacro:if>
   </joint>
   <link name="right_l2">
@@ -245,5 +277,7 @@
     <axis xyz="0 0 1"/>
     <limit effort="40.0" lower="-3.0426" upper="3.0426" velocity="1.957"/>
-    <dynamics damping="5.0" friction="5.0"/>
+<xacro:if value="$(arg gazebo)">
+    <dynamics damping="5.0" friction="2.0"/>
+</xacro:if>
   </joint>
   <link name="right_l3">
@@ -273,5 +307,7 @@
     <axis xyz="0 0 1"/>
     <limit effort="40.0" lower="-3.0439" upper="3.0439" velocity="1.957"/>
-    <dynamics damping="5.0" friction="5.0"/>
+ <xacro:if value="$(arg gazebo)">
+    <dynamics damping="15.0" friction="5.0"/>
+</xacro:if>
   </joint>
   <link name="right_l4">
@@ -301,5 +337,25 @@
     <axis xyz="0 0 1"/>
     <limit effort="9.0" lower="-2.9761" upper="2.9761" velocity="3.485"/>
-    <dynamics damping="2.0" friction="2.0"/>
+<xacro:if value="$(arg gazebo)">
+    <dynamics damping="30.0" friction="10.0"/>
+</xacro:if>
+  </joint>
+  <link name="right_arm_itb">
+<xacro:if value="$(arg gazebo)">
+    <xacro:gazebo_minimum_inertia />
+</xacro:if>
+<xacro:unless value="$(arg gazebo)">
+    <inertial>
+      <origin rpy="0 0 0" xyz="0.000000 0.000000 0.000000"/>
+      <mass value="0.0001"/>
+      <inertia ixx="1e-08" ixy="0" ixz="0" iyy="1e-08" iyz="0" izz="1e-08"/>
+    </inertial>
+</xacro:unless>
+  </link>
+  <joint name="right_arm_itb" type="fixed">
+    <origin rpy="0 -1.57079632679 0" xyz="-.055 0 .075"/>
+    <parent link="right_l4"/>
+    <child link="right_arm_itb"/>
+    <axis xyz="0 0 1"/>
   </joint>
   <link name="right_l5">
@@ -329,12 +385,12 @@
     <axis xyz="0 0 1"/>
     <limit effort="9.0" lower="-2.9761" upper="2.9761" velocity="3.485"/>
-    <dynamics damping="2.0" friction="2.0"/>
+<xacro:if value="$(arg gazebo)">
+    <dynamics damping="30.0" friction="10.0"/>
+</xacro:if>
   </joint>
   <link name="right_hand_camera">
-      <inertial>
-        <origin rpy="0 0 0" xyz="0 0 0"/>
-        <mass value="0.01"/>
-        <inertia ixx="0.1" ixy="0" ixz="0" iyy="0.1" iyz="0" izz="0.1"/>
-      </inertial>
+<xacro:if value="$(arg gazebo)">
+    <xacro:gazebo_minimum_inertia />
+</xacro:if>
   </link>
   <joint name="right_hand_camera" type="fixed">
@@ -345,9 +401,7 @@
   </joint>
   <link name="right_wrist">
-      <inertial>
-        <origin rpy="0 0 0" xyz="0 0 0"/>
-        <mass value="0.01"/>
-        <inertia ixx="0.1" ixy="0" ixz="0" iyy="0.1" iyz="0" izz="0.1"/>
-      </inertial>
+<xacro:if value="$(arg gazebo)">
+    <xacro:gazebo_minimum_inertia />
+</xacro:if>
   </link>
   <joint name="right_wrist" type="fixed">
@@ -382,7 +436,11 @@
     <child link="right_l6"/>
     <axis xyz="0 0 1"/>
-    <!-- limit effort="9.0" lower="-4.7124" upper="4.7124" velocity="4.545"/ -->
+<xacro:if value="$(arg gazebo)">
     <limit effort="9.0" lower="-3.14" upper="3.14" velocity="4.545"/>
-    <dynamics damping="2.0" friction="2.0"/>
+    <dynamics damping="30.0" friction="10.0"/>
+</xacro:if>
+<xacro:unless value="$(arg gazebo)">
+    <limit effort="9.0" lower="-4.7124" upper="4.7124" velocity="4.545"/>
+</xacro:unless>
   </joint>
   <link name="right_hand">
@@ -393,9 +451,14 @@
       </geometry>
     </collision>
-    <inertial>
-      <origin rpy="0 0 0" xyz="0 0 0"/>
-      <mass value="0.01"/>
-      <inertia ixx="0.1" ixy="0" ixz="0" iyy="0.1" iyz="0" izz="0.1"/>
-    </inertial>
+<xacro:if value="$(arg gazebo)">
+      <xacro:gazebo_minimum_inertia />
+</xacro:if>
+<xacro:unless value="$(arg gazebo)">
+    <inertial>
+      <origin rpy="0 0 0" xyz="1.0E-08 1.0E-08 1.0E-08"/>
+      <mass value="1.0E-08"/>
+      <inertia ixx="1.0E-08" ixy="1.0E-08" ixz="1.0E-08" iyy="1.0E-08" iyz="1.0E-08" izz="1.0E-08"/>
+    </inertial>
+</xacro:unless>
   </link>
   <joint name="right_hand" type="fixed">
@@ -404,5 +467,77 @@
     <parent link="right_l6"/>
     <child link="right_hand"/>
-</joint>
+  </joint>
+  <link name="right_l1_2">
+<xacro:if value="$(arg gazebo)">
+    <xacro:gazebo_minimum_inertia />
+</xacro:if>
+<xacro:unless value="$(arg gazebo)">
+    <inertial>
+      <origin rpy="0 0 0" xyz="1.0E-08 1.0E-08 1.0E-08"/>
+      <mass value="1.0E-08"/>
+      <inertia ixx="1.0E-08" ixy="1.0E-08" ixz="1.0E-08" iyy="1.0E-08" iyz="1.0E-08" izz="1.0E-08"/>
+    </inertial>
+</xacro:unless>
+    <collision>
+      <origin rpy="0 0 0" xyz="0 0 0.035"/>
+      <geometry>
+        <cylinder length="0.14" radius="0.07"/>
+      </geometry>
+    </collision>
+  </link>
+  <joint name="right_j1_2" type="fixed">
+    <origin rpy="0 0 0" xyz="0 0 0"/>
+    <parent link="right_l1"/>
+    <child link="right_l1_2"/>
+    <axis xyz="0 0 1"/>
+  </joint>
+  <link name="right_l2_2">
+<xacro:if value="$(arg gazebo)">
+    <xacro:gazebo_minimum_inertia />
+</xacro:if>
+<xacro:unless value="$(arg gazebo)">
+    <inertial>
+      <origin rpy="0 0 0" xyz="1.0E-08 1.0E-08 1.0E-08"/>
+      <mass value="1.0E-08"/>
+      <inertia ixx="1.0E-08" ixy="1.0E-08" ixz="1.0E-08" iyy="1.0E-08" iyz="1.0E-08" izz="1.0E-08"/>
+    </inertial>
+</xacro:unless>
+    <collision>
+      <origin rpy="0 0 0" xyz="0 0 0.26"/>
+      <geometry>
+        <sphere radius="0.06"/>
+      </geometry>
+    </collision>
+  </link>
+  <joint name="right_j2_2" type="fixed">
+    <origin rpy="0 0 0" xyz="0 0 0"/>
+    <parent link="right_l2"/>
+    <child link="right_l2_2"/>
+    <axis xyz="0 0 1"/>
+  </joint>
+  <link name="right_l4_2">
+<xacro:if value="$(arg gazebo)">
+    <xacro:gazebo_minimum_inertia />
+</xacro:if>
+<xacro:unless value="$(arg gazebo)">
+    <inertial>
+      <origin rpy="0 0 0" xyz="1.0E-08 1.0E-08 1.0E-08"/>
+      <mass value="1.0E-08"/>
+      <inertia ixx="1.0E-08" ixy="1.0E-08" ixz="1.0E-08" iyy="1.0E-08" iyz="1.0E-08" izz="1.0E-08"/>
+    </inertial>
+</xacro:unless>
+    <collision>
+      <origin rpy="0 0 0" xyz="0 0.01 0.26"/>
+      <geometry>
+        <sphere radius="0.06"/>
+      </geometry>
+    </collision>
+  </link>
+  <joint name="right_j4_2" type="fixed">
+    <origin rpy="0 0 0" xyz="0 0 0"/>
+    <parent link="right_l4"/>
+    <child link="right_l4_2"/>
+    <axis xyz="0 0 1"/>
+  </joint>
   <link name="screen">
     <visual>
@@ -419,9 +554,14 @@
       </geometry>
     </collision>
-    <inertial>
-      <origin rpy="0 0 0" xyz="0 0 0"/>
-      <mass value="0.01"/>
-      <inertia ixx="0.1" ixy="0" ixz="0" iyy="0.1" iyz="0" izz="0.1"/>
-    </inertial>
+<xacro:if value="$(arg gazebo)">
+    <xacro:gazebo_minimum_inertia />
+</xacro:if>
+<xacro:unless value="$(arg gazebo)">
+    <inertial>
+      <origin rpy="0 0 0" xyz="0 0 0"/>
+      <mass value="0.0001"/>
+      <inertia ixx="1e-08" ixy="0" ixz="0" iyy="1e-08" iyz="0" izz="1e-08"/>
+    </inertial>
+</xacro:unless>
   </link>
   <joint name="display_joint" type="fixed">
@@ -431,9 +571,7 @@
   </joint>
   <link name="head_camera">
-      <inertial>
-        <origin rpy="0 0 0" xyz="0 0 0"/>
-        <mass value="0.01"/>
-        <inertia ixx="0.1" ixy="0" ixz="0" iyy="0.1" iyz="0" izz="0.1"/>
-      </inertial>
+<xacro:if value="$(arg gazebo)">
+    <xacro:gazebo_minimum_inertia />
+</xacro:if>
   </link>
   <joint name="head_camera" type="fixed">

Commit message: Additional damping for j0 joint

File: sawyer_description/urdf/sawyer_base.urdf.xacro (robot description, xacro)
@@ -147,5 +147,5 @@
     <limit effort="80.0" lower="-3.0503" upper="3.0503" velocity="1.74"/>
 <xacro:if value="$(arg gazebo)">
-    <dynamics damping="5.0" friction="2.0"/>
+    <dynamics damping="10.0" friction="5.0"/>
 </xacro:if>
   </joint>
